File: power_switch.kicad_sch (KiCad schematic)
At the start: 16 parts, among them J1 Power Output, U1 BTS7004-1EPP

Commit message: use 1% resistor for voltage divider, add one more fiducial
Parts:
- R33: value 8.2kΩ -> 8.2kΩ 1%
- R35: value 1.8kΩ -> 1.8kΩ 1%
- R39: value 12kΩ -> 12kΩ 1%
Changed lines of the file:
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@@
       (effects (font (size 1.27 1.27)) (justify left))
     )
-    (property "Value" "8.2kΩ" (id 1) (at 80.01 52.07 0)
+    (property "Value" "8.2kΩ 1%" (id 1) (at 80.01 52.07 0)
       (effects (font (size 1.27 1.27)) (justify left))
     )
@@
       (effects (font (size 1.27 1.27)) (justify left))
     )
-    (property "Value" "1.8kΩ" (id 1) (at 80.01 77.47 0)
+    (property "Value" "1.8kΩ 1%" (id 1) (at 80.01 77.47 0)
       (effects (font (size 1.27 1.27)) (justify left))
     )
@@
     (in_bom yes) (on_board yes)
     (property "Reference" "R39" (id 0) (at 93.98 74.93 90))
-    (property "Value" "12kΩ" (id 1) (at 93.98 72.39 90))
+    (property "Value" "12kΩ 1%" (id 1) (at 93.98 72.39 90))
     (property "Footprint" "Resistor_SMD:R_0603_1608Metric" (id 2) (at 93.98 69.85 0)
       (effects (font (size 1.27 1.27)) hide)

Commit message: add uC controlled status LED, improve filling zones, move LED closer to connectors
Connections:
- net GND: now also D3.1 (K), D6.1 (K); no longer R13.1, R17.1
- net SW_FAULT: now also R17.2; no longer D6.2 (A)
- net SW_IN: now also R13.2; no longer D3.2 (A)
- new net: D6.2 (A), R17.1
- new net: D3.2 (A), R13.1
Other:
- moved on the sheet: D3, D6, R13, R17
Changed lines of the file:
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@@
   (paper "A4")
   (title_block
+    (date "2020-11-09")
+    (rev "v0.1")
     (comment 4 "Author: Stefan Agner")
   )
@@
   (symbol (lib_id "power:VDD") (at 93.98 29.21 0)
     (in_bom yes) (on_board yes)
-    (property "Reference" "#PWR044" (id 0) (at 93.98 33.02 0)
+    (property "Reference" "#PWR045" (id 0) (at 93.98 33.02 0)
       (effects (font (size 1.27 1.27)) hide)
     )
@@
   (symbol (lib_id "power:GND") (at 38.1 57.15 0)
     (in_bom yes) (on_board yes)
-    (property "Reference" "#PWR07" (id 0) (at 38.1 63.5 0)
+    (property "Reference" "#PWR09" (id 0) (at 38.1 63.5 0)
       (effects (font (size 1.27 1.27)) hide)
     )
@@
   (symbol (lib_id "power:GND") (at 57.15 57.15 0)
     (in_bom yes) (on_board yes)
-    (property "Reference" "#PWR018" (id 0) (at 57.15 63.5 0)
+    (property "Reference" "#PWR021" (id 0) (at 57.15 63.5 0)
       (effects (font (size 1.27 1.27)) hide)
     )
@@
   (symbol (lib_id "power:GND") (at 57.15 82.55 0)
     (in_bom yes) (on_board yes)
-    (property "Reference" "#PWR024" (id 0) (at 57.15 88.9 0)
+    (property "Reference" "#PWR023" (id 0) (at 57.15 88.9 0)
       (effects (font (size 1.27 1.27)) hide)
     )
@@
   (symbol (lib_id "power:GND") (at 57.15 124.46 0)
     (in_bom yes) (on_board yes)
-    (property "Reference" "#PWR026" (id 0) (at 57.15 130.81 0)
+    (property "Reference" "#PWR028" (id 0) (at 57.15 130.81 0)
       (effects (font (size 1.27 1.27)) hide)
     )
@@
   (symbol (lib_id "power:GND") (at 57.15 142.24 0)
     (in_bom yes) (on_board yes)
-    (property "Reference" "#PWR030" (id 0) (at 57.15 148.59 0)
+    (property "Reference" "#PWR032" (id 0) (at 57.15 148.59 0)
       (effects (font (size 1.27 1.27)) hide)
     )
@@
   (symbol (lib_id "power:GND") (at 77.47 57.15 0)
     (in_bom yes) (on_board yes)
-    (property "Reference" "#PWR035" (id 0) (at 77.47 63.5 0)
+    (property "Reference" "#PWR038" (id 0) (at 77.47 63.5 0)
       (effects (font (size 1.27 1.27)) hide)
     )
@@
   (symbol (lib_id "power:GND") (at 77.47 82.55 0)
     (in_bom yes) (on_board yes)
-    (property "Reference" "#PWR040" (id 0) (at 77.47 88.9 0)
+    (property "Reference" "#PWR041" (id 0) (at 77.47 88.9 0)
       (effects (font (size 1.27 1.27)) hide)
     )
@@
   (symbol (lib_id "power:GND") (at 93.98 57.15 0)
     (in_bom yes) (on_board yes)
-    (property "Reference" "#PWR048" (id 0) (at 93.98 63.5 0)
+    (property "Reference" "#PWR049" (id 0) (at 93.98 63.5 0)
       (effects (font (size 1.27 1.27)) hide)
     )
@@
   (symbol (lib_id "power:GND") (at 113.03 81.28 0)
     (in_bom yes) (on_board yes)
-    (property "Reference" "#PWR056" (id 0) (at 113.03 87.63 0)
+    (property "Reference" "#PWR054" (id 0) (at 113.03 87.63 0)
       (effects (font (size 1.27 1.27)) hide)
     )
@@
     )
     (property "Datasheet" "" (id 3) (at 113.03 81.28 0)
+      (effects (font (size 1.27 1.27)) hide)
+    )
+  )
+  (symbol (lib_id "Device:R_Small") (at 44.45 121.92 270)
+    (in_bom yes) (on_board yes)
+    (property "Reference" "R13" (id 0) (at 44.45 116.84 90))
+    (property "Value" "10kΩ" (id 1) (at 44.45 119.38 90))
+    (property "Footprint" "Resistor_SMD:R_0603_1608Metric" (id 2) (at 44.45 120.142 90)
+      (effects (font (size 1.27 1.27)) hide)
+    )
+    (property "Datasheet" "~" (id 3) (at 44.45 121.92 0)
+      (effects (font (size 1.27 1.27)) hide)
+    )
+  )
+  (symbol (lib_id "Device:R_Small") (at 44.45 139.7 270)
+    (in_bom yes) (on_board yes)
+    (property "Reference" "R17" (id 0) (at 44.45 134.62 90))
+    (property "Value" "10kΩ" (id 1) (at 44.45 137.16 90))
+    (property "Footprint" "Resistor_SMD:R_0603_1608Metric" (id 2) (at 44.45 137.922 90)
+      (effects (font (size 1.27 1.27)) hide)
+    )
+    (property "Datasheet" "~" (id 3) (at 44.45 139.7 0)
       (effects (font (size 1.27 1.27)) hide)
     )
@@
     )
   )
-  (symbol (lib_id "Device:R_Small") (at 52.07 121.92 270)
-    (in_bom yes) (on_board yes)
-    (property "Reference" "R13" (id 0) (at 52.07 116.84 90))
-    (property "Value" "10kΩ" (id 1) (at 52.07 119.38 90))
-    (property "Footprint" "Resistor_SMD:R_0603_1608Metric" (id 2) (at 52.07 120.142 90)
-      (effects (font (size 1.27 1.27)) hide)
-    )
-    (property "Datasheet" "~" (id 3) (at 52.07 121.92 0)
-      (effects (font (size 1.27 1.27)) hide)
-    )
-  )
-  (symbol (lib_id "Device:R_Small") (at 52.07 139.7 270)
-    (in_bom yes) (on_board yes)
-    (property "Reference" "R17" (id 0) (at 52.07 134.62 90))
-    (property "Value" "10kΩ" (id 1) (at 52.07 137.16 90))
-    (property "Footprint" "Resistor_SMD:R_0603_1608Metric" (id 2) (at 52.07 137.922 90)
-      (effects (font (size 1.27 1.27)) hide)
-    )
-    (property "Datasheet" "~" (id 3) (at 52.07 139.7 0)
-      (effects (font (size 1.27 1.27)) hide)
-    )
-  )
   (symbol (lib_id "Device:R_Small") (at 66.04 36.83 0)
     (in_bom yes) (on_board yes)
@@
     )
   )
-  (symbol (lib_id "Device:LED_Small") (at 44.45 121.92 0) (mirror y)
-    (in_bom yes) (on_board yes)
-    (property "Reference" "D3" (id 0) (at 44.45 115.57 0))
-    (property "Value" "GREEN" (id 1) (at 44.45 118.11 0))
-    (property "Footprint" "LED_SMD:LED_0603_1608Metric" (id 2) (at 44.45 121.92 90)
-      (effects (font (size 1.27 1.27)) hide)
-    )
-    (property "Datasheet" "~" (id 3) (at 44.45 121.92 90)
-      (effects (font (size 1.27 1.27)) hide)
-    )
-  )
-  (symbol (lib_id "Device:LED_Small") (at 44.45 139.7 0) (mirror y)
-    (in_bom yes) (on_board yes)
-    (property "Reference" "D6" (id 0) (at 44.45 133.35 0))
-    (property "Value" "RED" (id 1) (at 44.45 135.89 0))
-    (property "Footprint" "LED_SMD:LED_0603_1608Metric" (id 2) (at 44.45 139.7 90)
-      (effects (font (size 1.27 1.27)) hide)
-    )
-    (property "Datasheet" "~" (id 3) (at 44.45 139.7 90)
-      (effects (font (size 1.27 1.27)) hide)
-    )
+  (symbol (lib_id "Device:LED_Small") (at 52.07 121.92 0) (mirror y)
+    (in_bom yes) (on_board yes)
+    (property "Reference" "D3" (id 0) (at 52.07 115.57 0))
+    (property "Value" "GREEN" (id 1) (at 52.07 118.11 0))
+    (property "Footprint" "LED_SMD:LED_0603_1608Metric" (id 2) (at 52.07 121.92 90)
+      (effects (font (size 1.27 1.27)) hide)
+    )
+    (property "Datasheet" "~" (id 3) (at 52.07 121.92 90)
+      (effects (font (size 1.27 1.27)) hide)
+    )
+  )
+  (symbol (lib_id "Device:LED_Small") (at 52.07 139.7 0) (mirror y)
+    (in_bom yes) (on_board yes)
+    (property "Reference" "D6" (id 0) (at 52.07 133.35 0))
+    (property "Value" "RED" (id 1) (at 52.07 135.89 0))
+    (property "Footprint" "LED_SMD:LED_0603_1608Metric" (id 2) (at 52.07 139.7 90)
+      (effects (font (size 1.27 1.27)) hide)
+    )
+    (property "Datasheet" "~" (id 3) (at 52.07 139.7 90)
+      (effects (font (size 1.27 1.27)) hide)
+    )
